File: rangemaster-npnium/rangemaster.sch (KiCad schematic (older format))
At the start: 18 parts, among them J1 Conn_01x07_Male, Q1 Q_NPN_CBE

Commit message: Migrating transistor footprint
Parts:
- added TP1: Vb, TestPoint:TestPoint_THTPad_1.5x1.5mm_Drill0.7mm, symbol Connector:TestPoint
- Q1: footprint pedal-component-footprint:Transistor_KTYU-3-6_CBE_d11.7mm -> pedal-component-footprint:Transistor_TO-5_CBE_d10.1mm
Connections:
- net at C1.1, Q1.2 (B), R1.2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: now also TP1.1
Changed lines of the file:
@@
 F 0 "Q1" H 3391 5896 50  0000 L CNN
 F 1 "Q_NPN_CBE" H 3391 5805 50  0000 L CNN
-F 2 "pedal-component-footprint:Transistor_KTYU-3-6_CBE_d11.7mm" H 3400 5950 50  0001 C CNN
+F 2 "pedal-component-footprint:Transistor_TO-5_CBE_d10.1mm" H 3400 5950 50  0001 C CNN
 F 3 "~" H 3200 5850 50  0001 C CNN
 	1    3200 5850
@@
 	2650 5850 2650 5600
 Wire Wire Line
-	2200 5850 2650 5850
+	2200 5850 2450 5850
 Wire Wire Line
 	3300 5350 3300 5650
@@
 Wire Wire Line
 	1400 3650 1100 3650
+$Comp
+L Connector:TestPoint TP1
+U 1 1 6175E388
+P 2450 4650
+F 0 "TP1" H 2508 4768 50  0000 L CNN
+F 1 "Vb" H 2508 4677 50  0000 L CNN
+F 2 "TestPoint:TestPoint_THTPad_1.5x1.5mm_Drill0.7mm" H 2650 4650 50  0001 C CNN
+F 3 "~" H 2650 4650 50  0001 C CNN
+	1    2450 4650
+	1    0    0    -1
+$EndComp
+Wire Wire Line
+	2450 4650 2450 5850
+Connection ~ 2450 5850
+Wire Wire Line
+	2450 5850 2650 5850
 $EndSCHEMATC
