File: 3pdt-npnium/3pdt-npnium.kicad_pcb (KiCad board)
At the start: 2 copper layers, 19 x 30 mm, 3 parts, among them J1 PedalBoardHeader, SW1 pedalmarkt.com

Commit message: wip
Other:
- net class Default removed
- net class PWR removed
