File: fuzzface-npnium/fuzz-face.sch (KiCad schematic (older format))
At the start: 27 parts, among them Q1 Q_NPN_CBE, Q2 Q_NPN_CBE

Commit message: V2
Parts:
- Q1, Q2: footprint pedal-component-footprint:Transistor_KTYU-3-6_CBE_d11.7mm -> pedal-component-footprint:Transistor_TO-5_CBE_d10.1mm_2
Changed lines of the file:
@@
 F 0 "Q1" H 3291 4596 50  0000 L CNN
 F 1 "Q_NPN_CBE" H 3291 4505 50  0000 L CNN
-F 2 "pedal-component-footprint:Transistor_KTYU-3-6_CBE_d11.7mm" H 3300 4650 50  0001 C CNN
+F 2 "pedal-component-footprint:Transistor_TO-5_CBE_d10.1mm_2" H 3300 4650 50  0001 C CNN
 F 3 "~" H 3100 4550 50  0001 C CNN
 	1    3100 4550
@@
 F 0 "Q2" H 3941 4246 50  0000 L CNN
 F 1 "Q_NPN_CBE" H 3941 4155 50  0000 L CNN
-F 2 "pedal-component-footprint:Transistor_KTYU-3-6_CBE_d11.7mm" H 3950 4300 50  0001 C CNN
+F 2 "pedal-component-footprint:Transistor_TO-5_CBE_d10.1mm_2" H 3950 4300 50  0001 C CNN
 F 3 "~" H 3750 4200 50  0001 C CNN
 	1    3750 4200
@@
 P 1950 3650
 AR Path="/614076A9" Ref="#PWR?"  Part="1"
-AR Path="/6140A369/614076A9" Ref="#PWR?"  Part="1"
-F 0 "#PWR?" H 1950 3400 50  0001 C CNN
+AR Path="/6140A369/614076A9" Ref="#PWR0101"  Part="1"
+F 0 "#PWR0101" H 1950 3400 50  0001 C CNN
 F 1 "GND" H 1955 3477 50  0000 C CNN
 F 2 "" H 1950 3650 50  0001 C CNN

Commit message: wip
Parts:
- RV3: value 1K -> B1K
Changed lines of the file:
@@
 AR Path="/6140A369/61418BA7" Ref="RV3"  Part="1"
 F 0 "RV3" H 3780 5496 50  0000 R CNN
-F 1 "1K" H 3780 5405 50  0000 R CNN
+F 1 "B1K" H 3780 5405 50  0000 R CNN
 F 2 "MBv3 potentiometers:16MM_B.MOUNT_BANZAI" H 3850 5450 50  0001 C CNN
 F 3 "~" H 3850 5450 50  0001 C CNN
