File: fuzzface-npnium/npnium.kicad_pcb (KiCad board)
At the start: 2 copper layers, 58 x 42 mm, 35 parts, among them Q1 Q_NPN_CBE, Q2 Q_NPN_CBE

Commit message: V2
Parts:
- Q1, Q2: footprint pedal-component-footprint:Transistor_KTYU-3-6_CBE_d11.7mm -> pedal-component-footprint:Transistor_TO-5_CBE_d10.1mm_2
Routing:
- net Net-(C1-Pad1): track 22.3 -> 27.0 mm
- net Net-(Q1-Pad1): track 53.2 -> 49.5 mm
- net Net-(Q2-Pad1): track 14.5 -> 17.0 mm
Other:
- board text added: "&"
- board text added: "2"
- board text added: "v2"
- board text removed: "B u z z"
- board text removed: "Buzz Face v1"
- board text removed: "F a c e"

Commit message: wip
Parts:
- added G***: LOGO, graphics:pedalmarkt-logo-30x30, B.Cu at (100.8, 95.5)
Other:
- net class Default removed
- net class PWR removed
- board text added: "2&"
- board text removed: "&"
- board text removed: "2"
