File: fuzzface-npnium/fuzz-face.kicad_sch (KiCad schematic)
At the start: 27 parts, among them Q1 Q_NPN_CBE, Q2 Q_NPN_CBE

Commit message: JLC
Parts:
- removed H1, H5: GND, pedal-component-footprint:PinHeader_1x01_P2.54mm_Long_Front_Back, symbol Mechanical:MountingHole_Pad
- removed H10, H8: JACK_GND, pedal-component-footprint:PinHeader_1x01_P2.54mm_Long_Front_Back, symbol Mechanical:MountingHole_Pad
- removed H11, H15: LED+, pedal-component-footprint:PinHeader_1x01_P2.54mm_Long_Front_Back, symbol Mechanical:MountingHole_Pad
- removed H12: LED-, pedal-component-footprint:PinHeader_1x01_P2.54mm_Long_Front_Back, symbol Mechanical:MountingHole_Pad
- removed H13, H7: PEDAL_IN, pedal-component-footprint:PinHeader_1x01_P2.54mm_Long_Front_Back, symbol Mechanical:MountingHole_Pad
- removed H14, H9: PEDAL_OUT, pedal-component-footprint:PinHeader_1x01_P2.54mm_Long_Front_Back, symbol Mechanical:MountingHole_Pad
- removed H2, H6: 9V, pedal-component-footprint:PinHeader_1x01_P2.54mm_Long_Front_Back, symbol Mechanical:MountingHole_Pad
- removed H3: FX_IN, pedal-component-footprint:PinHeader_1x01_P2.54mm_Long_Front_Back, symbol Mechanical:MountingHole_Pad
- removed H4: FX_OUT, pedal-component-footprint:PinHeader_1x01_P2.54mm_Long_Front_Back, symbol Mechanical:MountingHole_Pad
- added D1: LED, LED_THT:LED_D5.0mm, symbol Device:LED
- added J1: +9v, Connector_JST:JST_XH_S2B-XH-A-1_1x02_P2.50mm_Horizontal, symbol Connector:Conn_01x02_Male
- added J2: Conn_01x06_Female, Connector_PinHeader_2.54mm:PinHeader_1x06_P2.54mm_Vertical, symbol Connector:Conn_01x06_Female
- added J4, J5: Conn_01x02_Female, Connector_PinHeader_2.54mm:PinHeader_1x02_P2.54mm_Vertical, symbol Connector:Conn_01x02_Female
- added R2: Rled, Resistor_THT:R_Axial_DIN0207_L6.3mm_D2.5mm_P7.62mm_Horizontal, symbol Device:R
- Q1, Q2: value Q_NPN_CBE -> Q_NPN_EBC; footprint pedal-component-footprint:Transistor_TO-5_CBE_d10.1mm_2 -> Package_TO_SOT_THT:TO-92L_Inline_Wide; symbol Device:Q_NPN_CBE -> Device:Q_NPN_EBC
- renumbered Cp1 to C4, R2 to R3
Connections:
- net +9V: now also J1.2 (Pin_2), R2.2
- net FX_IN: now also J2.2 (Pin_2)
- net FX_OUT: now also J2.6 (Pin_6)
- net GND: now also Q1.1 (E), J1.1 (Pin_1), J2.5 (Pin_5), J4.1 (Pin_1), J5.1 (Pin_1); no longer Q1.3 (E)
- net at Q2.2 (B), RV1.2, RV1.3: now also Q1.3 (C); no longer Q1.1 (C)
- net at RV2.2, RV2.3: now also Q2.3 (C); no longer Q2.1 (C)
- net at R1.1, RV3.3: now also Q2.1 (E); no longer Q2.3 (E)
- new net: D1.2 (A), R2.1
- new net IN: J2.1 (Pin_1), J4.2 (Pin_2)
- new net LED_GND: D1.1 (K), J2.3 (Pin_3)
- new net OUT: J2.4 (Pin_4), J5.2 (Pin_2)
