File: fuzzface-npnium/npnium-mainboard.kicad_pcb (KiCad board)
At the start: 2 copper layers, 58 x 80 mm, 58 parts, among them J1 +9v, J2 Conn_01x06_Female, J3 Conn_01x06_Female, J4 Conn_01x02_Female, J5 Conn_01x02_Female, Q1 Q_NPN_EBC, Q2 Q_NPN_EBC, SW1 SW_Push_3PDT

Commit message: JLC
Parts:
- removed J3: Conn_01x06_Female, Connector_PinHeader_2.54mm:PinHeader_1x06_P2.54mm_Vertical
- removed SW1: SW_Push_3PDT, pedal-component-footprint:3PDT.LUGS.FLPVSK
- removed the kibuzzard-6618FE8B at (93.6, 136.2)
- removed the kibuzzard-6618FE93 at (96.1, 135.6)
- removed the kibuzzard-6618FE9C at (98.7, 135.6)
- removed the kibuzzard-6618FEA0 at (101.2, 135.6)
- removed the kibuzzard-6618FEAA at (103.8, 135.6)
- removed the kibuzzard-6618FEB1 at (106.3, 135.6)
- removed kibuzzard-66194892: G***, kibuzzard-66194892
Routing:
- net /Switch/FX_OUT: track 38.6 -> 0.00 mm
- net /Switch/OUT: track 31.2 -> 0.00 mm
- net /Switch/LED_GND: track 22.5 -> 0.00 mm
- net /Switch/IN: track 20.4 -> 0.00 mm
- net /Switch/FX_IN: track 14.6 -> 0.00 mm
- net /Switch/GND: vias 6 -> 0
- removed copper zone on B.Cu, net /Switch/GND
- removed copper zone on F.Cu, net /Switch/GND
Other:
- board size 58 x 80 mm -> 58 x 42 mm
