File: fuzzface-npnium/npnium.kicad_sch (KiCad schematic)
At the start: 0 parts

Commit message: JLC
Other:
- added sheet Switch (switch.kicad_sch)
Changed lines of the file:
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@@
+    )
+  )
+  (sheet (at 17.78 39.37) (size 12.7 11.43) (fields_autoplaced)
+    (stroke (width 0.1524) (type solid) (color 0 0 0 0))
+    (fill (color 0 0 0 0.0000))
+    (property "Sheet name" "Switch" (id 0) (at 17.78 38.6584 0)
+      (effects (font (size 1.27 1.27)) (justify left bottom))
+    )
+    (property "Sheet file" "switch.kicad_sch" (id 1) (at 17.78 51.3846 0)
+      (effects (font (size 1.27 1.27)) (justify left top))
     )
   )
@@
     (path "/" (page "1"))
     (path "/00000000-0000-0000-0000-00006140a369" (page "2"))
+    (path "/f73370cd-c775-4b52-bc49-0fae253aa87d" (page "3"))
   )
   (symbol_instances
@@
       (reference "#PWR06") (unit 1) (value "+9V") (footprint "")
     )
-    (path "/00000000-0000-0000-0000-00006140a369/00000000-0000-0000-0000-00006140853b"
-      (reference "#PWR07") (unit 1) (value "+9V") (footprint "")
-    )
     (path "/00000000-0000-0000-0000-00006140a369/00000000-0000-0000-0000-000061418be0"
       (reference "#PWR08") (unit 1) (value "GND") (footprint "")
@@
       (reference "#PWR012") (unit 1) (value "GND") (footprint "")
     )
-    (path "/00000000-0000-0000-0000-00006140a369/00000000-0000-0000-0000-0000614076a9"
-      (reference "#PWR0101") (unit 1) (value "GND") (footprint "")
+    (path "/00000000-0000-0000-0000-00006140a369/7c0d126a-4c4b-47e2-8668-20b3dd22a8c8"
+      (reference "#PWR0101") (unit 1) (value "+9V") (footprint "")
     )
     (path "/00000000-0000-0000-0000-00006140a369/00000000-0000-0000-0000-0000613c96e3"
@@
     )
     (path "/00000000-0000-0000-0000-00006140a369/00000000-0000-0000-0000-000061418c03"
-      (reference "Cp1") (unit 1) (value "47u") (footprint "Capacitor_THT:CP_Radial_D5.0mm_P2.50mm")
+      (reference "C4") (unit 1) (value "47u") (footprint "Capacitor_THT:CP_Radial_D5.0mm_P2.50mm")
     )
-    (path "/00000000-0000-0000-0000-00006140a369/00000000-0000-0000-0000-0000613f4c20"
-      (reference "H1") (unit 1) (value "GND") (footprint "pedal-component-footprint:PinHeader_1x01_P2.54mm_Long_Front_Back")
+    (path "/00000000-0000-0000-0000-00006140a369/32b6260e-cfc7-4c90-8ad7-42255c880076"
+      (reference "D1") (unit 1) (value "LED") (footprint "LED_THT:LED_D5.0mm")
     )
-    (path "/00000000-0000-0000-0000-00006140a369/00000000-0000-0000-0000-0000613f6012"
-      (reference "H2") (unit 1) (value "9V") (footprint "pedal-component-footprint:PinHeader_1x01_P2.54mm_Long_Front_Back")
+    (path "/00000000-0000-0000-0000-00006140a369/a289ff88-d00c-4153-88d8-0aeb88171025"
+      (reference "J1") (unit 1) (value "+9v") (footprint "Connector_JST:JST_XH_S2B-XH-A-1_1x02_P2.50mm_Horizontal")
     )
-    (path "/00000000-0000-0000-0000-00006140a369/00000000-0000-0000-0000-0000613f6a38"
-      (reference "H3") (unit 1) (value "FX_IN") (footprint "pedal-component-footprint:PinHeader_1x01_P2.54mm_Long_Front_Back")
+    (path "/00000000-0000-0000-0000-00006140a369/f93b8c2e-ba7b-46d2-a521-694d2e1c1dfd"
+      (reference "J2") (unit 1) (value "Conn_01x06_Female") (footprint "Connector_PinHeader_2.54mm:PinHeader_1x06_P2.54mm_Vertical")
     )
-    (path "/00000000-0000-0000-0000-00006140a369/00000000-0000-0000-0000-0000613f6b94"
-      (reference "H4") (unit 1) (value "FX_OUT") (footprint "pedal-component-footprint:PinHeader_1x01_P2.54mm_Long_Front_Back")
+    (path "/f73370cd-c775-4b52-bc49-0fae253aa87d/3cb4a100-b0e3-4619-ae85-16f7de56df8e"
+      (reference "J3") (unit 1) (value "Conn_01x06_Female") (footprint "Connector_PinHeader_2.54mm:PinHeader_1x06_P2.54mm_Vertical")
     )
-    (path "/00000000-0000-0000-0000-00006140a369/00000000-0000-0000-0000-000061408542"
-      (reference "H5") (unit 1) (value "GND") (footprint "pedal-component-footprint:PinHeader_1x01_P2.54mm_Long_Front_Back")
+    (path "/00000000-0000-0000-0000-00006140a369/21c9094f-eb3c-45f9-aad3-2368045fddc2"
+      (reference "J4") (unit 1) (value "Conn_01x02_Female") (footprint "Connector_PinHeader_2.54mm:PinHeader_1x02_P2.54mm_Vertical")
     )
-    (path "/00000000-0000-0000-0000-00006140a369/00000000-0000-0000-0000-000061408548"
-      (reference "H6") (unit 1) (value "9V") (footprint "pedal-component-footprint:PinHeader_1x01_P2.54mm_Long_Front_Back")
-    )
-    (path "/00000000-0000-0000-0000-00006140a369/00000000-0000-0000-0000-00006140958a"
-      (reference "H7") (unit 1) (value "PEDAL_IN") (footprint "pedal-component-footprint:PinHeader_1x01_P2.54mm_Long_Front_Back")
-    )
-    (path "/00000000-0000-0000-0000-00006140a369/00000000-0000-0000-0000-00006141f531"
-      (reference "H8") (unit 1) (value "JACK_GND") (footprint "pedal-component-footprint:PinHeader_1x01_P2.54mm_Long_Front_Back")
-    )
-    (path "/00000000-0000-0000-0000-00006140a369/00000000-0000-0000-0000-00006141d1a2"
-      (reference "H9") (unit 1) (value "PEDAL_OUT") (footprint "pedal-component-footprint:PinHeader_1x01_P2.54mm_Long_Front_Back")
-    )
-    (path "/00000000-0000-0000-0000-00006140a369/00000000-0000-0000-0000-0000614232f8"
-      (reference "H10") (unit 1) (value "JACK_GND") (footprint "pedal-component-footprint:PinHeader_1x01_P2.54mm_Long_Front_Back")
-    )
-    (path "/00000000-0000-0000-0000-00006140a369/00000000-0000-0000-0000-00006142eff3"
-      (reference "H11") (unit 1) (value "LED+") (footprint "pedal-component-footprint:PinHeader_1x01_P2.54mm_Long_Front_Back")
-    )
-    (path "/00000000-0000-0000-0000-00006140a369/00000000-0000-0000-0000-000061430bd3"
-      (reference "H12") (unit 1) (value "LED-") (footprint "pedal-component-footprint:PinHeader_1x01_P2.54mm_Long_Front_Back")
-    )
-    (path "/00000000-0000-0000-0000-00006140a369/00000000-0000-0000-0000-00006140a915"
-      (reference "H13") (unit 1) (value "PEDAL_IN") (footprint "pedal-component-footprint:PinHeader_1x01_P2.54mm_Long_Front_Back")
-    )
-    (path "/00000000-0000-0000-0000-00006140a369/00000000-0000-0000-0000-00006141d1a8"
-      (reference "H14") (unit 1) (value "PEDAL_OUT") (footprint "pedal-component-footprint:PinHeader_1x01_P2.54mm_Long_Front_Back")
-    )
-    (path "/00000000-0000-0000-0000-00006140a369/00000000-0000-0000-0000-00006142f6d9"
-      (reference "H15") (unit 1) (value "LED+") (footprint "pedal-component-footprint:PinHeader_1x01_P2.54mm_Long_Front_Back")
+    (path "/00000000-0000-0000-0000-00006140a369/b5206845-f29b-428c-9d9d-c46eadda8381"
+      (reference "J5") (unit 1) (value "Conn_01x02_Female") (footprint "Connector_PinHeader_2.54mm:PinHeader_1x02_P2.54mm_Vertical")
     )
     (path "/00000000-0000-0000-0000-00006140a369/00000000-0000-0000-0000-000061418b82"
-      (reference "Q1") (unit 1) (value "Q_NPN_CBE") (footprint "pedal-component-footprint:Transistor_TO-5_CBE_d10.1mm_2")
+      (reference "Q1") (unit 1) (value "Q_NPN_EBC") (footprint "Package_TO_SOT_THT:TO-92L_Inline_Wide")
     )
     (path "/00000000-0000-0000-0000-00006140a369/00000000-0000-0000-0000-000061418b88"
-      (reference "Q2") (unit 1) (value "Q_NPN_CBE") (footprint "pedal-component-footprint:Transistor_TO-5_CBE_d10.1mm_2")
+      (reference "Q2") (unit 1) (value "Q_NPN_EBC") (footprint "Package_TO_SOT_THT:TO-92L_Inline_Wide")
     )
     (path "/00000000-0000-0000-0000-00006140a369/00000000-0000-0000-0000-000061418b97"
       (reference "R1") (unit 1) (value "100K") (footprint "Resistor_THT:R_Axial_DIN0207_L6.3mm_D2.5mm_P7.62mm_Horizontal")
     )
+    (path "/00000000-0000-0000-0000-00006140a369/c1d63bb8-7310-4a19-8ba3-42817d61c7ab"
+      (reference "R2") (unit 1) (value "Rled") (footprint "Resistor_THT:R_Axial_DIN0207_L6.3mm_D2.5mm_P7.62mm_Horizontal")
+    )
     (path "/00000000-0000-0000-0000-00006140a369/00000000-0000-0000-0000-000061418bcd"
-      (reference "R2") (unit 1) (value "470") (footprint "Resistor_THT:R_Axial_DIN0207_L6.3mm_D2.5mm_P7.62mm_Horizontal")
+      (reference "R3") (unit 1) (value "470") (footprint "Resistor_THT:R_Axial_DIN0207_L6.3mm_D2.5mm_P7.62mm_Horizontal")
     )
     (path "/00000000-0000-0000-0000-00006140a369/00000000-0000-0000-0000-000061418b8e"
@@
       (reference "RV4") (unit 1) (value "A500K") (footprint "MBv3 potentiometers:16MM_B.MOUNT_BANZAI")
     )
+    (path "/f73370cd-c775-4b52-bc49-0fae253aa87d/587daa46-34b0-4a21-9bcd-5e21c0978a48"
+      (reference "SW1") (unit 1) (value "SW_Push_3PDT") (footprint "pedal-component-footprint:3PDT.LUGS.FLPVSK")
+    )
   )
